File: hard/GPduinoWiFi/GPduinoWiFi.sch (EAGLE design)
At the start: 30 parts, among them CN1 EH-2, CN10 cn6, CN11 FTDI Basic, CN2 EH-2, CN3 PH-2, CN4 EH-4, CN5 PICOBLADE-3, CN6 PICOBLADE-3, CN7 PICOBLADE-3, CN8 cn6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

Commit message: ・回路図の修正（リビジョン番号のみ）
Other:
- note added: "2"
- note removed: "1"
Changed lines of the file:
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@@
 <text x="33.02" y="135.89" size="2.54" layer="97">Motor L</text>
 <text x="303.022" y="12.954" size="2.54" layer="94">Bizan Nishimura (@lipoyang)</text>
-<text x="376.174" y="21.336" size="2.54" layer="94">1</text>
+<text x="376.174" y="21.336" size="2.54" layer="94">2</text>
 <text x="212.09" y="135.89" size="2.54" layer="97">2 type connectors</text>
 <text x="33.02" y="88.9" size="2.54" layer="97">Motor R</text>
